File: PCBbasics.kicad_pcb (KiCad board)
At the start: 2 copper layers, 24 parts, among them SW1 SW_Push, U1 ATmega32U4-A, Y1 16MHz

Commit message: PCB Finished
Parts:
- C5, C7, U1: moved to B.Cu
- USB1: footprint random-keyboard-parts:PJ-3200B-4A-Assembly -> random-keyboard-parts:Molex-0548190589
- moved R2 88.3 mm to (111.9, 136.3), turned to 90 degrees
- moved SW1 72.2 mm to (124.5, 148.2)
- moved C7 63.8 mm to (146.8, 146.8), turned to 180 degrees
- moved U1 62.6 mm to (142.1, 134.9)
- moved R3 54.6 mm to (116.7, 136.3), turned to -90 degrees
- moved USB1 53.2 mm to (113.5, 117.6), turned to -90 degrees
- moved C2 51.4 mm to (150.0, 119.9), turned to -90 degrees
- moved C6 50.2 mm to (138.1, 146.8)
- moved R1 49.0 mm to (131.8, 128.8), turned to 90 degrees
- moved F1 48.9 mm to (124.4, 127.8)
- moved C4 45.7 mm to (153.2, 138.8), turned to 90 degrees
- moved R4 44.6 mm to (158.8, 134.1), turned to -90 degrees
- moved C1 37.1 mm to (134.1, 119.9), turned to 90 degrees
- moved C3 36.8 mm to (128.6, 135.1), turned to -90 degrees
- moved C5 36.8 mm to (153.2, 131.0), turned to 90 degrees
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Other:
- board outline added: 98.4 x 38.1 mm
